Commit message: Fixed

File: description/robot_core.xacro (robot description, xacro)
@@ -28,5 +28,5 @@
             <origin xyz="0.15 0 0.075" rpy="0 0 0" />
             <geometry>
-                <box size="0.3 0.3 0.15" />
+                <mesh> <uri> model://description/meshes/chassis.stl</uri> </mesh>
             </geometry>
             <material name="white" />
@@ -35,5 +35,5 @@
             <origin xyz="0.15 0 0.075" rpy="0 0 0" />
             <geometry>
-                <box size="0.3 0.3 0.15" />
+                <mesh> <uri> model://description/meshes/chassis.stl</uri> </mesh>
             </geometry>
         </collision>
@@ -44,4 +44,7 @@
     <gazebo reference="chasis">
         <material>Gazebo/White</material>
+        <geometry>
+            <mesh> <uri> model://description/meshes/chassis.stl</uri> </mesh>
+        </geometry>
     </gazebo>
     <!-- LEFT WHEEL -->
