Commit message: Revert "Fixed"

File: src/description/robot_core.xacro (robot description, xacro)
@@ -28,5 +28,5 @@
             <origin xyz="0.15 0 0.075" rpy="0 0 0" />
             <geometry>
-                <mesh> <uri> model://description/meshes/chassis.stl</uri> </mesh>
+                <box size="0.3 0.3 0.15" />
             </geometry>
             <material name="white" />
@@ -35,5 +35,5 @@
             <origin xyz="0.15 0 0.075" rpy="0 0 0" />
             <geometry>
-                <mesh> <uri> model://description/meshes/chassis.stl</uri> </mesh>
+                <box size="0.3 0.3 0.15" />
             </geometry>
         </collision>
@@ -44,7 +44,4 @@
     <gazebo reference="chasis">
         <material>Gazebo/White</material>
-        <geometry>
-            <mesh> <uri> model://description/meshes/chassis.stl</uri> </mesh>
-        </geometry>
     </gazebo>
     <!-- LEFT WHEEL -->

Commit message: got gz to load stl by adding stl to ./gazebo/model

File: src/description/robot_core.xacro (robot description, xacro)
@@ -28,5 +28,5 @@
             <origin xyz="0.15 0 0.075" rpy="0 0 0" />
             <geometry>
-                <box size="0.3 0.3 0.15" />
+                <mesh filename="package://jbot2/description/meshes/chassis.stl" scale="0.001 0.001 0.001" />
             </geometry>
             <material name="white" />
@@ -35,5 +35,6 @@
             <origin xyz="0.15 0 0.075" rpy="0 0 0" />
             <geometry>
-                <box size="0.3 0.3 0.15" />
+                <mesh filename="package://jbot2/description/meshes/chassis.stl" scale="0.001 0.001 0.001"/>
+                <!-- <box size="0.3 0.3 0.15" /> -->
             </geometry>
         </collision>
@@ -42,6 +43,9 @@
         </xacro:inertial_box>
     </link>
-    <gazebo reference="chasis">
+    <gazebo reference="chassis">
         <material>Gazebo/White</material>
+        <geometry>
+            <mesh package="$(find jbot2)/description/meshes/chassis.stl" scale="0.001 0.001 0.001"/>
+        </geometry>
     </gazebo>
     <!-- LEFT WHEEL -->
